File: pullup_counter_schematic/pullup_counter_schematic.kicad_pcb (KiCad board)
At the start: 2 copper layers, 97 x 65 mm, 69 parts, among them J1 USB_B_Micro, J2 6PinDebugPort, J3 Micro_SD_Card, Q1 MMBT3904, SW1 boot, SW2 rst, SW3 UsrBtn0, SW4 start, SW5 UsrBtn1, SW6 UsrBtn2, SW7 UsrBtn3, U1 MT3608, U2 STM32G070RBT6, U3 CH340C, U4 ITR8307, U5 W25Q80, Y1 32.768KHz, Y2 8MHz

Commit message: Minor fixes
Changed lines of the file:
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@@
   (net 12 "/OSC_OUT")
   (net 13 "Net-(C20-Pad1)")
-  (net 14 "Net-(C21-Pad1)")
+  (net 14 "Net-(DS1-Pad28)")
   (net 15 "Net-(D1-Pad2)")
   (net 16 "/SCK")
@@
     (fp_line (start -1 0.625) (end -1 -0.625) (layer "F.Fab") (width 0.1))
     (pad "1" smd roundrect (at -1.0375 0 180) (size 1.175 1.45) (layers "F.Cu" "F.Paste" "F.Mask") (roundrect_rratio 0.212766)
-      (net 14 "Net-(C21-Pad1)") (pintype "passive"))
+      (net 14 "Net-(DS1-Pad28)") (pintype "passive"))
     (pad "2" smd roundrect (at 1.0375 0 180) (size 1.175 1.45) (layers "F.Cu" "F.Paste" "F.Mask") (roundrect_rratio 0.212766)
       (net 1 "GND") (pintype "passive"))
@@
     (property "Sheetname" "")
     (attr through_hole)
-    (fp_text reference "TP1" (at 0.8 -2.4) (layer "F.SilkS")
+    (fp_text reference "TP1" (at -0.05 -2.05) (layer "F.SilkS")
       (effects (font (size 1 1) (thickness 0.15)))
     )
@@
     (property "Sheetname" "")
     (attr through_hole)
-    (fp_text reference "TP2" (at 0 -2.77) (layer "F.SilkS")
+    (fp_text reference "TP2" (at 0 -2.2) (layer "F.SilkS")
       (effects (font (size 1 1) (thickness 0.15)))
     )
@@
       (net 13 "Net-(C20-Pad1)") (pinfunction "VCOMH") (pintype "passive"))
     (pad "28" smd rect (at -8.75 0) (size 0.4 2) (layers "B.Cu" "B.Paste" "B.Mask")
-      (net 14 "Net-(C21-Pad1)") (pinfunction "VCC") (pintype "power_in"))
+      (net 14 "Net-(DS1-Pad28)") (pinfunction "VCC") (pintype "power_in"))
     (pad "29" smd rect (at -9.45 0) (size 0.4 2) (layers "B.Cu" "B.Paste" "B.Mask")
       (net 1 "GND") (pinfunction "VLSS") (pintype "power_in"))
@@
   (via (at 105.1 93.8) (size 0.9) (drill 0.4) (layers "F.Cu" "B.Cu") (free) (net 1))
   (via (at 116.9 46.9) (size 0.9) (drill 0.4) (layers "F.Cu" "B.Cu") (free) (net 1))
-  (via (at 164 41.2) (size 0.9) (drill 0.4) (layers "F.Cu" "B.Cu") (free) (net 1))
+  (via (at 164 42.25) (size 0.9) (drill 0.4) (layers "F.Cu" "B.Cu") (free) (net 1))
   (via (at 173.5 56.7) (size 0.6) (drill 0.3) (layers "F.Cu" "B.Cu") (free) (net 1))
   (via (at 143.2 46.3) (size 0.6) (drill 0.3) (layers "F.Cu" "B.Cu") (free) (net 1))
@@
   (segment (start 130.2 59.7) (end 128.2 61.7) (width 0.2) (layer "B.Cu") (net 42))
   (segment (start 132.8 59.7) (end 130.2 59.7) (width 0.2) (layer "B.Cu") (net 42))
+  (segment (start 158.1 42.1) (end 157.1 41.1) (width 0.2) (layer "F.Cu") (net 45))
   (segment (start 112.55 45.05) (end 116.5 41.1) (width 0.2) (layer "F.Cu") (net 45))
-  (segment (start 157.7 42.1) (end 156.7 41.1) (width 0.2) (layer "F.Cu") (net 45))
-  (segment (start 161.65 42.1) (end 157.7 42.1) (width 0.2) (layer "F.Cu") (net 45))
+  (segment (start 161.65 42.1) (end 158.1 42.1) (width 0.2) (layer "F.Cu") (net 45))
+  (segment (start 157.1 41.1) (end 156.7 41.1) (width 0.2) (layer "F.Cu") (net 45))
   (segment (start 112.55 49.38) (end 112.55 45.05) (width 0.2) (layer "F.Cu") (net 45))
   (via (at 156.7 41.1) (size 0.6) (drill 0.3) (layers "F.Cu" "B.Cu") (net 45))
@@
   (segment (start 156.7 41.1) (end 116.5 41.1) (width 0.2) (layer "B.Cu") (net 45))
   (segment (start 113.65 45.15) (end 116.9 41.9) (width 0.2) (layer "F.Cu") (net 46))
-  (segment (start 157.4 42.6) (end 156.7 41.9) (width 0.2) (layer "F.Cu") (net 46))
+  (segment (start 161.65 42.6) (end 157.85 42.6) (width 0.2) (layer "F.Cu") (net 46))
   (segment (start 113.65 49.38) (end 113.65 45.15) (width 0.2) (layer "F.Cu") (net 46))
-  (segment (start 161.65 42.6) (end 157.4 42.6) (width 0.2) (layer "F.Cu") (net 46))
+  (segment (start 157.15 41.9) (end 156.7 41.9) (width 0.2) (layer "F.Cu") (net 46))
+  (segment (start 157.85 42.6) (end 157.15 41.9) (width 0.2) (layer "F.Cu") (net 46))
   (via (at 116.9 41.9) (size 0.6) (drill 0.3) (layers "F.Cu" "B.Cu") (net 46))
   (via (at 156.7 41.9) (size 0.6) (drill 0.3) (layers "F.Cu" "B.Cu") (net 46))
   (segment (start 156.7 41.9) (end 116.9 41.9) (width 0.2) (layer "B.Cu") (net 46))
-  (segment (start 157.1 43.1) (end 156.7 42.7) (width 0.2) (layer "F.Cu") (net 47))
+  (segment (start 160.84467 43.1) (end 160.74467 43) (width 0.2) (layer "F.Cu") (net 47))
+  (segment (start 157.684314 43) (end 157.384314 42.7) (width 0.2) (layer "F.Cu") (net 47))
+  (segment (start 160.74467 43) (end 157.684314 43) (width 0.2) (layer "F.Cu") (net 47))
+  (segment (start 157.384314 42.7) (end 156.7 42.7) (width 0.2) (layer "F.Cu") (net 47))
   (segment (start 115.85 49.38) (end 115.85 45.35) (width 0.2) (layer "F.Cu") (net 47))
   (segment (start 115.85 45.35) (end 118.5 42.7) (width 0.2) (layer "F.Cu") (net 47))
-  (segment (start 161.65 43.1) (end 157.1 43.1) (width 0.2) (layer "F.Cu") (net 47))
+  (segment (start 161.65 43.1) (end 160.84467 43.1) (width 0.2) (layer "F.Cu") (net 47))
   (via (at 156.7 42.7) (size 0.6) (drill 0.3) (layers "F.Cu" "B.Cu") (net 47))
   (via (at 118.5 42.7) (size 0.6) (drill 0.3) (layers "F.Cu" "B.Cu") (net 47))

Commit message: Generated gerbers for hardware V03
Other:
- board text added: "JLCJLCJLCJLC"
Changed lines of the file:
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@@
+    (effects (font (size 0.8128 0.8128) (thickness 0.1524)))
+  )
+  (gr_text "JLCJLCJLCJLC" (at 140.2 62.6) (layer "F.SilkS")
     (effects (font (size 0.8128 0.8128) (thickness 0.1524)))
   )
